File: Modular_hat_in_out_kicad/Modular_hat_in_out.kicad_pcb (KiCad board)
At the start: 2 copper layers, 65 x 56 mm, 150 parts, among them J1 Raspberry_Pi_2_3, U1 MCP3008, U2 LM324, U3 MCP3008, U4 MCP4728, U5 MCP4728, U6 LM324

Commit message: [ADD] Somes pigeons
Parts:
- added REF**: Pigeon-6, Modular Shield:Pigeon-6, B.Cu at (42.1, 49.5)
- added REF**: Pigeon-5, Modular Shield:Pigeon-5, B.Cu at (53.0, 60.6)
- added REF**: Pigeon-4, Modular Shield:Pigeon-4, B.Cu at (32.5, 60.4)
- turned REF** to 0 degrees (x2)

Commit message: [ADD] 2 Metalic pigeons
Parts:
- moved REF** 1.97 mm to (53.0, 58.7)
- moved REF** 1.97 mm to (32.5, 58.5)

Commit message: [ADD] One more metalic pigeon
Parts:
- turned REF** to 180 degrees

Commit message: [ADD] Pigeon citation
Other:
- board text added: "Pigeons Gobble Up Soft Bread"
