File: Modular_hat_in_out_kicad/Modular_hat_in_out.kicad_sch (KiCad schematic)
At the start: 65 parts, among them J1 Raspberry_Pi_2_3, U1 MCP3008, U2 LM324, U3 MCP3008, U4 MCP4728, U5 MCP4728, U6 LM324

Commit message: [ADD] Update to last kicad version
Other:
- moved on the sheet: J1, JP1, JP2, JP4, JP5, JP7, JP8

Commit message: [ADD] Footprints
Parts:
- C1, C2, C3, C4: footprint (none) -> Modular Shield:C_0603_1608Metric
- U4, U5: footprint Package_SO:MSOP-10_3x3mm_P0.5mm -> Modular Shield:MCP4728 MSOP10
Changed lines of the file:
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@@
 			)
 		)
-		(property "Footprint" ""
+		(property "Footprint" "Modular Shield:C_0603_1608Metric"
 			(at 260.6548 119.38 0)
 			(effects
@@
 			)
 		)
-		(property "Footprint" "Package_SO:MSOP-10_3x3mm_P0.5mm"
+		(property "Footprint" "Modular Shield:MCP4728 MSOP10"
 			(at 198.12 115.57 0)
 			(effects
@@
 			)
 		)
-		(property "Description" ""
+		(property "Description" "12-bit digital to analog converter, quad output, 2.048V internal reference, integrated EEPROM, I2C interface"
 			(at 198.12 134.62 0)
 			(effects
@@
 			)
 		)
-		(property "Footprint" ""
+		(property "Footprint" "Modular Shield:C_0603_1608Metric"
 			(at 203.5048 119.38 0)
 			(effects
@@
 			)
 		)
-		(property "Footprint" ""
+		(property "Footprint" "Modular Shield:C_0603_1608Metric"
 			(at 272.0848 119.38 0)
 			(effects
@@
 			)
 		)
-		(property "Footprint" ""
+		(property "Footprint" "Modular Shield:C_0603_1608Metric"
 			(at 192.0748 119.38 0)
 			(effects
@@
 			)
 		)
-		(property "Footprint" "Package_SO:MSOP-10_3x3mm_P0.5mm"
+		(property "Footprint" "Modular Shield:MCP4728 MSOP10"
 			(at 267.97 115.57 0)
 			(effects
@@
 			)
 		)
-		(property "Description" ""
+		(property "Description" "12-bit digital to analog converter, quad output, 2.048V internal reference, integrated EEPROM, I2C interface"
 			(at 267.97 134.62 0)
 			(effects

Commit message: [ADD] LCSC Capacitor parts
Parts:
- C1, C3: LCSC (none) -> C14663
- C2, C4: LCSC (none) -> C1691
Changed lines of the file:
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@@
+			)
+		)
+		(property "LCSC" "C14663"
+			(at 261.62 123.19 0)
+			(effects
+				(font
+					(size 1.27 1.27)
+				)
+				(hide yes)
 			)
 		)
@@
 			)
 		)
+		(property "LCSC" "C1691"
+			(at 204.47 123.19 0)
+			(effects
+				(font
+					(size 1.27 1.27)
+				)
+				(hide yes)
+			)
+		)
 		(pin "1"
 		)
@@
 			)
 		)
+		(property "LCSC" "C1691"
+			(at 273.05 123.19 0)
+			(effects
+				(font
+					(size 1.27 1.27)
+				)
+				(hide yes)
+			)
+		)
 		(pin "1"
 		)
@@
 			(at 193.04 123.19 0)
 			(effects
+				(font
+					(size 1.27 1.27)
+				)
+				(hide yes)
+			)
+		)
+		(property "LCSC" "C14663"
+			(at 193.04 123.19 0)
+			(effects

Commit message: [ADD] ML324 footprint
Parts:
- U2, U6: footprint (none) -> Modular Shield:LM324 SOIC14; LCSC (none) -> C71035
Changed lines of the file:
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@@
 			)
 		)
-		(property "Footprint" ""
+		(property "Footprint" "Modular Shield:LM324 SOIC14"
 			(at 201.93 76.2 0)
 			(effects
@@
 		)
 		(property "Description" ""
+			(at 205.74 76.2 0)
+			(effects
+				(font
+					(size 1.27 1.27)
+				)
+				(hide yes)
+			)
+		)
+		(property "LCSC" "C71035"
 			(at 205.74 76.2 0)
 			(effects
@@
 			)
 		)
-		(property "Footprint" ""
+		(property "Footprint" "Modular Shield:LM324 SOIC14"
 			(at 201.93 35.56 0)
 			(effects
@@
 			(at 205.74 35.56 0)
 			(effects
+				(font
+					(size 1.27 1.27)
+				)
+				(hide yes)
+			)
+		)
+		(property "LCSC" "C71035"
+			(at 205.74 35.56 0)
+			(effects

Commit message: [ADD] 12V input in shematics
Parts:
- removed TP1, TP3: LDAC, symbol Modular Shield:TestPoint
- removed TP2, TP4, TP5, TP6: RDY, symbol Modular Shield:TestPoint
- added JP9: PINHD-1X2, Modular Shield:1X06-BIG, symbol Modular Shield:PINHD-1X2
Connections:
- net GND: now also JP9.2
- net GPIO25: now reaches J1.22 (GPIO25)
- net GPIO25: now also U4.5 (RDY/~{BSY})
- net GPIO0: now reaches J1.27 (ID_SD/GPIO0)
- net GPIO0: now also U4.4 (~{LDAC})
- net GPIO1: now reaches J1.28 (ID_SC/GPIO1)
- net GPIO1: now also U5.4 (~{LDAC})
- net GPIO20: now reaches J1.40 (GPIO21/SCLK1)
- net GPIO20: now also U5.5 (RDY/~{BSY})
- net +12V: now reaches U6.4 (VCC+)
- net +12V: now also U2.4 (VCC+), JP9.1
- no-connect marks 13 -> 9
Other:
- note added: "Input Voltage"
- note removed: "12V"
- note removed: "Test Points"

Commit message: [ADD] All components routed
Parts:
- JP9: footprint Modular Shield:1X06-BIG -> Modular Shield:1X02-BIG
Changed lines of the file:
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@@
 			)
 		)
-		(property "Footprint" "Modular Shield:1X06-BIG"
+		(property "Footprint" "Modular Shield:1X02-BIG"
 			(at 278.13 87.63 0)
 			(effects

Commit message: [ADD] Build for production
Parts:
- H1, H2, H3, H4, J1, JP1, JP2, JP3, JP4, JP5, JP6, JP7, JP8, JP9: now not fitted
- R59, R60, R63, R66, R76, R81, R83, R88: value 48K -> 43K; LCSC C227922 -> C23172
- U1, U3: JLCPCB Position Offset 0.65, 0 -> 0, -0.16
- U2, U6: JLCPCB Rotation Offset (none) -> 270
Changed lines of the file:
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@@
 		(in_bom no)
 		(on_board yes)
-		(dnp no)
+		(dnp yes)
 		(property "Reference" "JP4"
 			(at 114.3 19.685 0)
@@
 		(in_bom no)
 		(on_board yes)
-		(dnp no)
+		(dnp yes)
 		(property "Reference" "JP3"
 			(at 137.16 53.975 0)
@@
 		(in_bom no)
 		(on_board yes)
-		(dnp no)
+		(dnp yes)
 		(property "Reference" "H1"
 			(at 278.257 47.8536 0)
@@
 		(in_bom no)
 		(on_board yes)
-		(dnp no)
+		(dnp yes)
 		(property "Reference" "H2"
 			(at 278.257 52.9336 0)
@@
 		(in_bom no)
 		(on_board yes)
-		(dnp no)
+		(dnp yes)
 		(property "Reference" "H3"
 			(at 278.257 58.0136 0)
@@
 		(in_bom no)
 		(on_board yes)
-		(dnp no)
+		(dnp yes)
 		(property "Reference" "H4"
 			(at 278.257 63.0936 0)
@@
 			)
 		)
-		(property "JLCPCB Position Offset" "0.65, 0"
+		(property "JLCPCB Position Offset" "0, -0.16"
 			(at 269.24 175.26 0)
 			(effects
@@
 			)
 		)
-		(property "JLCPCB Position Offset" "0.65, 0"
+		(property "JLCPCB Position Offset" "0, -0.16"
 			(at 219.71 175.26 0)
 			(effects
@@
 		(in_bom no)
 		(on_board yes)
-		(dnp no)
+		(dnp yes)
 		(property "Reference" "J1"
 			(at 43.18 25.4 0)
@@
 		(in_bom no)
 		(on_board yes)
-		(dnp no)
+		(dnp yes)
 		(property "Reference" "JP6"
 			(at 137.16 19.685 0)
@@
 		(in_bom no)
 		(on_board yes)
-		(dnp no)
+		(dnp yes)
 		(property "Reference" "JP1"
 			(at 114.3 53.975 0)
@@
 		(in_bom no)
 		(on_board yes)
-		(dnp no)
+		(dnp yes)
 		(property "Reference" "JP5"
 			(at 114.3 88.265 0)
@@
 		(in_bom no)
 		(on_board yes)
-		(dnp no)
+		(dnp yes)
 		(property "Reference" "JP2"
 			(at 137.16 88.265 0)
@@
 			)
 		)
-		(property "Value" "48K"
+		(property "Value" "43K"
 			(at 179.07 25.4 90)
 			(effects
@@
 			)
 		)
-		(property "LCSC" "C227922"
+		(property "LCSC" "C23172"
 			(at 179.07 21.59 90)
 			(effects
@@
 		(in_bom no)
 		(on_board yes)
-		(dnp no)
+		(dnp yes)
 		(property "Reference" "JP7"
 			(at 114.3 125.095 0)
@@
 		(in_bom yes)
 		(on_board yes)
-		(dnp no)
+		(dnp yes)
 		(fields_autoplaced yes)
 		(property "Reference" "JP9"
@@
 			)
 		)
-		(property "Value" "48K"
+		(property "Value" "43K"
 			(at 179.07 66.04 90)
 			(effects
@@
 			)
 		)
-		(property "LCSC" "C227922"
+		(property "LCSC" "C23172"
 			(at 179.07 62.23 90)
 			(effects
@@
 			)
 		)
-		(property "Value" "48K"
+		(property "Value" "43K"
 			(at 232.41 25.4 90)
 			(effects
@@
 			)
 		)
-		(property "LCSC" "C227922"
+		(property "LCSC" "C23172"
 			(at 232.41 21.59 90)
 			(effects
@@
 			)
 		)
+		(property "JLCPCB Rotation Offset" "270"
+			(at 205.74 76.2 0)
+			(effects
+				(font
+					(size 1.27 1.27)
+				)
+				(hide yes)
+			)
+		)
 		(pin "1"
 		)
@@
 		(in_bom no)
 		(on_board yes)
-		(dnp no)
+		(dnp yes)
 		(property "Reference" "JP8"
 			(at 137.16 125.095 0)
@@
 			)
 		)
-		(property "Value" "48K"
+		(property "Value" "43K"
 			(at 179.07 93.98 90)
 			(effects
@@
 			)
 		)
-		(property "LCSC" "C227922"
+		(property "LCSC" "C23172"
 			(at 179.07 97.79 90)
 			(effects
@@
 			)
 		)
-		(property "Value" "48K"
+		(property "Value" "43K"
 			(at 232.41 53.34 90)
 			(effects
@@
 			)
 		)
-		(property "LCSC" "C227922"
+		(property "LCSC" "C23172"
 			(at 232.41 57.15 90)
 			(effects
@@
 			)
 		)
-		(property "Value" "48K"
+		(property "Value" "43K"
 			(at 232.41 93.98 90)
 			(effects
@@
 			)
 		)
-		(property "LCSC" "C227922"
+		(property "LCSC" "C23172"
 			(at 232.41 97.79 90)
 			(effects
@@
 			)
 		)
-		(property "Value" "48K"
+		(property "Value" "43K"
 			(at 179.07 53.34 90)
 			(effects
@@
 			)
 		)
-		(property "LCSC" "C227922"
+		(property "LCSC" "C23172"
 			(at 179.07 57.15 90)
 			(effects
@@
 			)
 		)
+		(property "JLCPCB Rotation Offset" "270"
+			(at 205.74 35.56 0)
+			(effects
+				(font
+					(size 1.27 1.27)
+				)
+				(hide yes)
+			)
+		)
 		(pin "1"
 		)
@@
 			)
 		)
-		(property "Value" "48K"
+		(property "Value" "43K"
 			(at 232.41 66.04 90)
 			(effects
@@
 			)
 		)
-		(property "LCSC" "C227922"
+		(property "LCSC" "C23172"
 			(at 232.41 62.23 90)
 			(effects

Commit message: [ADD] Revision number (1.0)
Other:
- title: (none) -> Modular Hat
Changed lines of the file:
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@@
 	(generator_version "8.0")
 	(paper "User" 317.627 242.138)
+	(title_block
+		(title "Modular Hat")
+		(date "2024-08-21")
+		(rev "1.0")
+	)
 	(junction
 		(at 242.57 137.16)
