File: Modular_hat_in_out_kicad/inputRegulator.kicad_sch (KiCad schematic)
At the start: 4 parts

Commit message: [ADD] Footprints
Parts:
- D3: footprint Modular Shield:D_0603_1608Metric -> Modular Shield:D_Z_0603_1608Metric
Changed lines of the file:
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@@
 			)
 		)
-		(property "Footprint" "Modular Shield:D_0603_1608Metric"
+		(property "Footprint" "Modular Shield:D_Z_0603_1608Metric"
 			(at 67.31 40.64 0)
 			(effects

Commit message: [ADD] Build for production
Parts:
- D1: renamed from D3; value D_Zener 6.6V -> D_Zener 6.8V; LCSC C894569 -> C2832575
- renumbered R8 to R1, R9 to R2, R10 to R3
Changed lines of the file:
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@@
 		(on_board yes)
 		(dnp no)
-		(property "Reference" "R9"
+		(property "Reference" "R2"
 			(at 72.39 30.48 90)
 			(effects
@@
 		(on_board yes)
 		(dnp no)
-		(property "Reference" "R10"
+		(property "Reference" "R3"
 			(at 82.55 30.48 90)
 			(effects
@@
 		(on_board yes)
 		(dnp no)
-		(property "Reference" "R8"
+		(property "Reference" "R1"
 			(at 62.23 30.48 90)
 			(effects
@@
 		(on_board yes)
 		(dnp no)
-		(property "Reference" "D3"
+		(property "Reference" "D1"
 			(at 67.31 46.99 0)
 			(effects
@@
 			)
 		)
-		(property "Value" "D_Zener 6.6V"
+		(property "Value" "D_Zener 6.8V"
 			(at 67.31 44.45 0)
 			(effects
@@
 			)
 		)
-		(property "LCSC" "C894569"
+		(property "LCSC" "C2832575"
 			(at 67.31 46.99 0)
 			(effects

Commit message: [ADD] Revision number (1.0)
Other:
- title: (none) -> Input Regulator
Changed lines of the file:
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@@
 	(generator_version "8.0")
 	(paper "User" 132.004 99.9998)
+	(title_block
+		(title "Input Regulator")
+		(date "2024-08-21")
+		(rev "1.0")
+	)
 	(junction
 		(at 55.88 33.02)
